File: kicad/testshield/testshield.kicad_pcb (KiCad board)
At the start: 2 copper layers, 26.7 x 55.9 mm, 6 parts, among them J1 ISP header, J2 Raspiheader, SW1 SW_Push, U1 ATMEGA328P-PU

Commit message: update
Parts:
- R1: footprint Resistors_THT:R_Axial_DIN0207_L6.3mm_D2.5mm_P10.16mm_Horizontal -> Resistors_SMD:R_2010
- U1: footprint ATMEGA328P-PU:DIP794W46P254L2967H457Q28B -> ATMEGA328P-AU:QFP80P900X900X120-32N
- moved J1 45.0 mm to (94.0, 87.6)
- moved SW1 44.2 mm to (91.4, 128.3)
- moved C1 35.9 mm to (87.6, 115.6), turned to 270 degrees
- moved R1 26.1 mm to (94.0, 115.6), turned to 270 degrees
- moved J2 16.5 mm to (101.6, 85.1)
- moved U1 15.3 mm to (91.4, 102.9), turned to 270 degrees
Routing:
- net +3V3: track 93.9 -> 46.4 mm
- net GNDD: track 102.5 -> 127.2 mm
- net Net-(J1-Pad3): track 17.4 -> 31.5 mm
- net Net-(J1-Pad1): track 13.8 -> 0.00 mm
- net Net-(J1-Pad4): track 16.4 -> 29.1 mm
- net Net-(SW1-Pad1): track 17.7 -> 8.64 mm
- net Net-(J2-Pad5): track 9.79 -> 16.4 mm
- net Net-(J2-Pad3): track 16.2 -> 21.3 mm
- added copper zone on F.Cu, net GNDD
Other:
- board size 26.7 x 55.9 mm -> 22.9 x 53.3 mm

Commit message: Add files via upload
Parts:
- removed J1: ISP header, Pin_Headers:Pin_Header_Straight_2x03_Pitch2.54mm
- removed R1: 10k, Resistors_SMD:R_2010
- removed SW1: SW_Push, Buttons_Switches_SMD:SW_SPST_B3S-1000
- moved U1 7.88 mm to (91.3, 95.0), turned to 0 degrees
- moved C1 5.78 mm to (88.5, 109.9), turned to 0 degrees
- moved J2 4.19 mm to (102.6, 81.0)
Connections:
- J2 pad 1: +3V3 -> Net-(J2-Pad1)
- J2 pad 14: Net-(J2-Pad14) -> GNDD
- J2 pad 17: Net-(J2-Pad17) -> +3V3
- J2 pad 20: Net-(J2-Pad20) -> GNDD
- J2 pad 25: Net-(J2-Pad25) -> GNDD
- J2 pad 30: Net-(J2-Pad30) -> GNDD
- J2 pad 34: Net-(J2-Pad34) -> GNDD
- J2 pad 39: Net-(J2-Pad39) -> GNDD
- J2 pad 9: Net-(J2-Pad9) -> GNDD
- U1 pad 1: Net-(SW1-Pad1) -> Net-(J2-Pad26)
- U1 pad 16: Net-(U1-Pad16) -> Net-(J2-Pad24)
- U1 pad 17: Net-(J1-Pad4) -> Net-(J2-Pad19)
- U1 pad 18: Net-(J1-Pad1) -> Net-(J2-Pad21)
- U1 pad 19: Net-(J1-Pad3) -> Net-(J2-Pad23)
- U1 pad 2: Net-(U1-Pad2) -> Net-(J2-Pad8)
- U1 pad 26: Net-(U1-Pad26) -> Net-(J2-Pad11)
- U1 pad 3: Net-(U1-Pad3) -> Net-(J2-Pad10)
- U1 pad 5: Net-(U1-Pad5) -> Net-(J2-Pad32)
Routing:
- net GNDD: track 127.2 -> 37.3 mm
- net Net-(J2-Pad26): track 0.00 -> 65.0 mm, vias 0 -> 2
- net Net-(J2-Pad10): track 0.00 -> 47.3 mm
- net Net-(J2-Pad32): track 0.00 -> 42.3 mm
- net Net-(J2-Pad8): track 0.00 -> 35.5 mm
- net Net-(J1-Pad3): track 31.5 -> 0.00 mm
- net Net-(J1-Pad4): track 29.1 -> 0.00 mm
- net Net-(J2-Pad23): track 0.00 -> 24.7 mm
- net Net-(J2-Pad24): track 0.00 -> 16.6 mm
- net Net-(J2-Pad21): track 0.00 -> 13.3 mm, vias 0 -> 2
- net Net-(J2-Pad11): track 0.00 -> 12.0 mm
- net Net-(J2-Pad19): track 0.00 -> 10.4 mm
- net +3V3: track 46.4 -> 36.8 mm
- net Net-(SW1-Pad1): track 8.64 -> 0.00 mm
- net Net-(J2-Pad3): track 21.3 -> 17.4 mm
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Other:
- board size 22.9 x 53.3 mm -> 27.8 x 59.7 mm
- board text added: "*"

Commit message: Add files via upload
Parts:
- added D1: LED1, LEDs:LED_0603, F.Cu at (144.0, 130.6)
- added D2: LED2, LEDs:LED_0603, F.Cu at (142.0, 130.6)
- added J1: ISP/PDI, Pin_Headers:Pin_Header_Straight_2x03_Pitch2.54mm, F.Cu at (147.3, 144.8)
- added R1: 1k, Resistors_SMD:R_0603, F.Cu at (144.0, 127.3)
- added R2: 330, Resistors_SMD:R_0603, F.Cu at (142.0, 105.4)
- added R3: 330, Resistors_SMD:R_0603, F.Cu at (142.0, 127.3)
- added R4: 10k, Resistors_SMD:R_0603, F.Cu at (146.1, 127.3)
- added SW1: Reset, Buttons_Switches_SMD:SW_SPST_B3U-1000P, F.Cu at (143.8, 100.3)
- moved C1 57.9 mm to (146.3, 106.2), turned to 90 degrees
- moved U1 56.3 mm to (143.0, 117.3), turned to 270 degrees
- moved J2 55.3 mm to (154.9, 99.1)
Routing:
- net +3V3: track 36.8 -> 159.5 mm
- net GNDD: track 37.3 -> 128.9 mm, vias 0 -> 1
- net Net-(J1-Pad5): track 65.0 -> 15.2 mm, vias 2 -> 0
- net Net-(J1-Pad1): track 13.3 -> 61.7 mm, vias 2 -> 0
- net Net-(J2-Pad10): track 47.3 -> 0.00 mm
- net Net-(J2-Pad32): track 42.3 -> 0.00 mm
- net Net-(J2-Pad8): track 35.5 -> 0.00 mm
- net Net-(J2-Pad5): track 13.5 -> 35.7 mm
- net Net-(J2-Pad24): track 16.6 -> 0.00 mm
- net Net-(J1-Pad4): track 10.4 -> 0.00 mm
- net Net-(R2-Pad2): track 0.00 -> 6.44 mm
- net Net-(D1-Pad2): track 0.00 -> 4.17 mm
- net Net-(J2-Pad3): track 17.4 -> 21.0 mm
- net Net-(D2-Pad2): track 0.00 -> 1.75 mm
- net Net-(J1-Pad3): track 24.7 -> 25.3 mm
- removed copper zone on F.Cu, net GNDD
Other:
- board outline removed
- board text removed: "*"

Commit message: pcb layout WIP
Parts:
- added R5: 2K7, Resistors_SMD:R_0603, F.Cu at (160.0, 105.4)
- added R6: 2K7, Resistors_SMD:R_0603, F.Cu at (162.6, 105.4)
- C1: footprint Capacitors_SMD:CP_Elec_3x5.3 -> Capacitors_SMD:c_elec_4x5.3
- D1, D2: footprint LEDs:LED_0603 -> LEDs:LED_0805
- J1: footprint Pin_Headers:Pin_Header_Straight_2x03_Pitch2.54mm -> Pin_Headers:Pin_Header_Straight_2x03
- J2: footprint Pin_Headers:Pin_Header_Straight_2x20_Pitch2.54mm -> Pin_Headers:Pin_Header_Straight_2x20
- SW1: footprint Buttons_Switches_SMD:SW_SPST_B3U-1000P -> Buttons_Switches_SMD:SW_SPST_B3SL-1022P
- moved R1 25.7 mm to (156.2, 149.9), turned to 0 degrees
- moved D1 25.1 mm to (160.0, 149.9), turned to 180 degrees
- moved D2 24.6 mm to (160.0, 147.3), turned to 180 degrees
- moved R3 24.6 mm to (156.2, 147.3), turned to 0 degrees
- moved R4 20.9 mm to (157.5, 144.8), turned to 0 degrees
- moved C1 19.6 mm to (134.6, 121.9), turned to 0 degrees
- moved SW1 12.3 mm to (154.9, 105.4), turned to 270 degrees
- moved U1 12.0 mm to (154.9, 118.1)
- moved J2 11.7 mm to (166.4, 101.6)
- moved R2 8.27 mm to (149.9, 108.0), turned to 90 degrees
- moved J1 6.35 mm to (152.4, 141.0), turned to 90 degrees
Connections:
- net Net-(J1-Pad1) renamed /MISO
- net Net-(J1-Pad3) renamed /SCK
- net Net-(J1-Pad4) renamed /MOSI
- net Net-(J1-Pad5) renamed /RST
- net Net-(J2-Pad10) renamed /RX
- net Net-(J2-Pad11) renamed /GPIO17
- net Net-(J2-Pad24) renamed /SS
- net Net-(J2-Pad3) renamed /SDA
- net Net-(J2-Pad5) renamed /SCL
- net Net-(J2-Pad8) renamed /TX
- J2 pad 1: Net-(J2-Pad1) -> +3V3
- J2 pad 12: Net-(J2-Pad12) -> /PWM
- J2 pad 16: Net-(J2-Pad16) -> /GPIO23
- U1 pad 24: Net-(U1-Pad24) -> /PWM
- U1 pad 25: Net-(U1-Pad25) -> /GPIO23
- U1 pad 5: Net-(J2-Pad32) -> Net-(U1-Pad5)
Routing:
- net +3V3: track 159.5 -> 6.42 mm
- net GNDD: track 128.9 -> 40.3 mm, vias 1 -> 0
- net /SCL: track 35.7 -> 0.00 mm
- net /MOSI: track 0.00 -> 33.7 mm, vias 0 -> 1
- net /SS: track 0.00 -> 26.0 mm, vias 0 -> 2
- net /MISO: track 61.7 -> 36.5 mm, vias 0 -> 2
- net /SDA: track 21.0 -> 0.00 mm
- net /PWM: track 0.00 -> 20.0 mm
- net /SCK: track 25.3 -> 37.5 mm
- net /GPIO23: track 0.00 -> 11.5 mm
- net Net-(R2-Pad2): track 6.44 -> 0.00 mm
- net Net-(D1-Pad2): track 4.17 -> 0.00 mm
- net /RST: track 15.2 -> 19.2 mm
- net /GPIO17: track 11.7 -> 9.72 mm
Other:
- net class Default: trace_width 0.25 -> 0.3; via_dia 0.6 -> 1.1; via_drill 0.4 -> 1

Commit message: pcb routes WIP
Parts:
- added H1: MountingHole_2.2mm_M2_ISO14580_Pad, Mounting_Holes:MountingHole_2.2mm_M2_ISO14580_Pad, F.Cu at (175.3, 95.2)
- added H2: MountingHole_2.2mm_M2_ISO14580_Pad, Mounting_Holes:MountingHole_2.2mm_M2_ISO14580_Pad, F.Cu at (175.3, 156.2)
- added H3: MountingHole_2.2mm_M2_ISO14580_Pad, Mounting_Holes:MountingHole_2.2mm_M2_ISO14580_Pad, F.Cu at (146.1, 156.2)
- added H4: MountingHole_2.2mm_M2_ISO14580_Pad, Mounting_Holes:MountingHole_2.2mm_M2_ISO14580_Pad, F.Cu at (146.1, 95.2)
- moved C1 23.9 mm to (156.2, 132.1), turned to 180 degrees
- moved R2 5.24 mm to (151.1, 113.0)
- moved U1 2.54 mm to (154.9, 120.7)
- moved J1 1.27 mm to (153.7, 141.0)
Routing:
- net +3V3: track 6.42 -> 102.0 mm
- net GNDD: track 40.3 -> 135.8 mm
- net /RST: track 19.2 -> 84.2 mm
- net /SS: track 26.0 -> 60.9 mm, vias 2 -> 0
- net /SDA: track 0.00 -> 31.9 mm
- net /RX: track 0.00 -> 25.8 mm, vias 0 -> 1
- net /SCL: track 0.00 -> 22.1 mm
- net /TX: track 0.00 -> 16.8 mm, vias 0 -> 1
- net /MOSI: track 33.7 -> 50.5 mm
- net Net-(R2-Pad2): track 0.00 -> 10.5 mm
- net /SCK: track 37.5 -> 43.4 mm
- net /GPIO17: track 9.72 -> 13.0 mm
- net /PWM: track 20.0 -> 22.7 mm
- net /MISO: track 36.5 -> 38.6 mm, vias 2 -> 0
- net Net-(D1-Pad2): track 0.00 -> 2.01 mm
Other:
- board outline added: 34.3 x 66 mm
- net class Default: via_dia 1.1 -> 1.5

Commit message: pcb layout done
v1.0
Parts:
- added G***: LOGO, testshield:bulldog_logo_smaller, F.Cu at (161.3, 128.3)
- moved C1 1.27 mm to (156.2, 133.3)
- moved H1 0.63 mm to (174.6, 95.2)
- moved H2 0.63 mm to (174.6, 156.2)
Routing:
- net +3V3: track 102.0 -> 108.7 mm
- net /SDA: track 31.9 -> 36.2 mm
- net /TX: track 16.8 -> 19.5 mm
- net /SCL: track 22.1 -> 24.8 mm
- net /SS: track 60.9 -> 62.5 mm
- net /RST: track 84.2 -> 84.7 mm
- added copper zone on B.Cu, net GNDD
- added copper zone on F.Cu, net GNDD
Other:
- board size 34.3 x 66 mm -> 33.7 x 66 mm
- board text added: "."
