File: kicad/testshield/testshield.kicad_pcb (KiCad board)
At the start: 2 copper layers, 33.7 x 66 mm, 22 parts, among them J1 ISP/PDI, J2 Raspiheader, SW1 Reset, U1 ATMEGA328P-AU

Commit message: created layout PDFs
Parts:
- moved R4 47.8 mm to (161.6, 101.6), turned to 180 degrees
- moved C1 0.69 mm to (155.4, 134.6)
- moved G*** 0.38 mm to (159.8, 128.9), turned to 270 degrees
Connections:
- J2 pad 12: /PWM -> /PWMp
- J2 pad 13: Net-(J2-Pad13) -> (no net)
- J2 pad 15: Net-(J2-Pad15) -> (no net)
- J2 pad 16: /GPIO23 -> /PWMa
- J2 pad 18: Net-(J2-Pad18) -> (no net)
- J2 pad 2: Net-(J2-Pad2) -> (no net)
- J2 pad 22: Net-(J2-Pad22) -> (no net)
- J2 pad 27: Net-(J2-Pad27) -> (no net)
- J2 pad 28: Net-(J2-Pad28) -> (no net)
- J2 pad 29: Net-(J2-Pad29) -> (no net)
- J2 pad 31: Net-(J2-Pad31) -> (no net)
- J2 pad 32: Net-(J2-Pad32) -> (no net)
- J2 pad 33: Net-(J2-Pad33) -> (no net)
- J2 pad 35: Net-(J2-Pad35) -> (no net)
- J2 pad 36: Net-(J2-Pad36) -> (no net)
- J2 pad 37: Net-(J2-Pad37) -> (no net)
- J2 pad 38: Net-(J2-Pad38) -> (no net)
- J2 pad 4: Net-(J2-Pad4) -> (no net)
- J2 pad 40: Net-(J2-Pad40) -> (no net)
- J2 pad 7: Net-(J2-Pad7) -> (no net)
- U1 pad 1: Net-(U1-Pad1) -> /PWMa
- U1 pad 10: Net-(U1-Pad10) -> (no net)
- U1 pad 11: Net-(U1-Pad11) -> (no net)
- U1 pad 13: Net-(U1-Pad13) -> (no net)
- U1 pad 19: Net-(U1-Pad19) -> (no net)
- U1 pad 2: Net-(U1-Pad2) -> (no net)
- U1 pad 22: Net-(U1-Pad22) -> (no net)
- U1 pad 23: Net-(U1-Pad23) -> (no net)
- U1 pad 24: /PWM -> (no net)
- U1 pad 25: /GPIO23 -> /PWMp
- U1 pad 32: Net-(U1-Pad32) -> (no net)
- U1 pad 7: Net-(U1-Pad7) -> (no net)
- U1 pad 8: Net-(U1-Pad8) -> (no net)
- U1 pad 9: Net-(U1-Pad9) -> (no net)
Routing:
- net /RST: track 132.6 -> 99.5 mm
- net /PWM: track 22.7 -> 0.00 mm
- net /PWMa: track 0.00 -> 16.2 mm, vias 0 -> 1
- net /PWMp: track 0.00 -> 14.8 mm
- net GNDD: track 132.3 -> 118.9 mm, vias 1 -> 0
- net +3V3: track 148.5 -> 160.8 mm
- net /GPIO23: track 11.4 -> 0.00 mm
- net /SS: track 28.6 -> 25.9 mm
- net /LED: track 36.4 -> 35.2 mm
- net /RX: track 16.0 -> 14.8 mm
- net /MOSI: track 38.3 -> 37.5 mm
- net /MISO: track 35.5 -> 34.9 mm
Other:
- board size 33.7 x 66 mm -> 32.4 x 66 mm
